Commit message: add gripper control

File: block.urdf (robot description, URDF)
Before this commit: robot block_2, 1 links, 0 joints
Links:
- link block_2_base_link: geometry collision box size=0.10 0.018 0.05; visual box size=0.10 0.018 0.05

Commit message: significant change on trajectory planning

File: block.urdf (robot description, URDF)
Before this commit: robot block_2, 1 links, 0 joints
Links:
- link block_2_base_link: geometry collision box size=0.30 0.018 0.05; visual box size=0.30 0.018 0.05
